File: PCB/makropad.kicad_sch (KiCad schematic)
At the start: 62 parts, among them J1 OLED_DISPLAY, J2 Conn_01x04, SW1 SW_Push_45deg, SW10 SW_Push_45deg, SW11 RotaryEncoder_Switch, SW12 RotaryEncoder_Switch, SW2 SW_Push_45deg, SW3 SW_Push_45deg, SW4 SW_Push_45deg, SW5 SW_Push_45deg, SW6 SW_Push_45deg, SW7 SW_Push_45deg, SW8 SW_Push_45deg, SW9 SW_Push_45deg, U1 PCF8574A, U2 MOUDLE-SEEEDUINO-XIAO

Commit message: fix some stuff + firmware
Connections:
- net COL0: now also SW11.S1; no longer SW12.S1
- net COL3: now also SW12.S1; no longer SW11.S1
- net ENC_1_SWA: now also D9.2 (A); no longer D12.2 (A)
- net ENC_2_SWA: now also D12.2 (A); no longer D9.2 (A)
- net ROW0: now also U2.11 (PA6_A10_D10_MOSI); no longer U2.10 (PA5_A9_D9_MISO)
- net ROW1: now also U2.10 (PA5_A9_D9_MISO); no longer U2.11 (PA6_A10_D10_MOSI)

Commit message: feat: switch to choc v2 switches
Parts:
- D23, D24, D25, D26, D27, D28: footprint LED_SMD:LED_SK6812MINI_PLCC4_3.5x3.5mm_P1.75mm -> Components:LED_SK6812MINI_PLCC4_3.5x3.5mm_P1.75mm
- SW1, SW10, SW2, SW3, SW4, SW5, SW6, SW7, SW8, SW9: footprint Components:Gateron Low Profile Switch 2.0 -> Components:SW_Kailh_Choc_V2
Changed lines of the file:
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@@
 		)
 	)
-	(global_label "RGB"
-		(shape input)
-		(at 24.13 121.92 180)
-		(fields_autoplaced yes)
-		(effects
-			(font
-				(size 1.27 1.27)
-			)
-			(justify right)
-		)
-		(property "Intersheetrefs" "${INTERSHEET_REFS}"
-			(at 17.3348 121.92 0)
-			(effects
-				(font
-					(size 1.27 1.27)
-				)
-				(justify right)
-				(hide yes)
-			)
-		)
-	)
 	(global_label "COL2"
 		(shape input)
@@
 		)
 	)
+	(global_label "RGB"
+		(shape input)
+		(at 24.13 121.92 180)
+		(fields_autoplaced yes)
+		(effects
+			(font
+				(size 1.27 1.27)
+			)
+			(justify right)
+		)
+		(property "Intersheetrefs" "${INTERSHEET_REFS}"
+			(at 17.3348 121.92 0)
+			(effects
+				(font
+					(size 1.27 1.27)
+				)
+				(justify right)
+				(hide yes)
+			)
+		)
+	)
 	(global_label "ENC_2_SWA"
 		(shape input)
@@
 			)
 		)
-		(property "Footprint" "LED_SMD:LED_SK6812MINI_PLCC4_3.5x3.5mm_P1.75mm"
+		(property "Footprint" "Components:LED_SK6812MINI_PLCC4_3.5x3.5mm_P1.75mm"
 			(at 186.69 157.48 0)
 			(effects
@@
 			)
 		)
-		(property "Footprint" "Components:Gateron Low Profile Switch 2.0"
+		(property "Footprint" "Components:SW_Kailh_Choc_V2"
 			(at 67.31 44.45 0)
 			(effects
@@
 			)
 		)
-		(property "Footprint" "Components:Gateron Low Profile Switch 2.0"
+		(property "Footprint" "Components:SW_Kailh_Choc_V2"
 			(at 92.71 44.45 0)
 			(effects
@@
 			)
 		)
-		(property "Footprint" "Components:Gateron Low Profile Switch 2.0"
+		(property "Footprint" "Components:SW_Kailh_Choc_V2"
 			(at 120.65 36.83 0)
 			(effects
@@
 			)
 		)
-		(property "Footprint" "LED_SMD:LED_SK6812MINI_PLCC4_3.5x3.5mm_P1.75mm"
+		(property "Footprint" "Components:LED_SK6812MINI_PLCC4_3.5x3.5mm_P1.75mm"
 			(at 171.45 157.48 0)
 			(effects
@@
 			)
 		)
-		(property "Footprint" "Components:Gateron Low Profile Switch 2.0"
+		(property "Footprint" "Components:SW_Kailh_Choc_V2"
 			(at 96.52 36.83 0)
 			(effects
@@
 			)
 		)
-		(property "Footprint" "Components:Gateron Low Profile Switch 2.0"
+		(property "Footprint" "Components:SW_Kailh_Choc_V2"
 			(at 71.12 36.83 0)
 			(effects
@@
 			)
 		)
-		(property "Footprint" "LED_SMD:LED_SK6812MINI_PLCC4_3.5x3.5mm_P1.75mm"
+		(property "Footprint" "Components:LED_SK6812MINI_PLCC4_3.5x3.5mm_P1.75mm"
 			(at 156.21 157.48 0)
 			(effects
@@
 			)
 		)
-		(property "Footprint" "Components:Gateron Low Profile Switch 2.0"
+		(property "Footprint" "Components:SW_Kailh_Choc_V2"
 			(at 116.84 44.45 0)
 			(effects
@@
 			)
 		)
-		(property "Footprint" "Components:Gateron Low Profile Switch 2.0"
+		(property "Footprint" "Components:SW_Kailh_Choc_V2"
 			(at 50.8 36.83 0)
 			(effects
@@
 			)
 		)
-		(property "Footprint" "LED_SMD:LED_SK6812MINI_PLCC4_3.5x3.5mm_P1.75mm"
+		(property "Footprint" "Components:LED_SK6812MINI_PLCC4_3.5x3.5mm_P1.75mm"
 			(at 186.69 129.54 0)
 			(effects
@@
 			)
 		)
-		(property "Footprint" "Components:Gateron Low Profile Switch 2.0"
+		(property "Footprint" "Components:SW_Kailh_Choc_V2"
 			(at 63.5 50.8 0)
 			(effects
@@
 			)
 		)
-		(property "Footprint" "LED_SMD:LED_SK6812MINI_PLCC4_3.5x3.5mm_P1.75mm"
+		(property "Footprint" "Components:LED_SK6812MINI_PLCC4_3.5x3.5mm_P1.75mm"
 			(at 171.45 129.54 0)
 			(effects
@@
 			)
 		)
-		(property "Footprint" "Components:Gateron Low Profile Switch 2.0"
+		(property "Footprint" "Components:SW_Kailh_Choc_V2"
 			(at 46.99 44.45 0)
 			(effects
@@
 			)
 		)
-		(property "Footprint" "Components:Gateron Low Profile Switch 2.0"
+		(property "Footprint" "Components:SW_Kailh_Choc_V2"
 			(at 88.9 50.8 0)
 			(effects
@@
 			)
 		)
-		(property "Footprint" "LED_SMD:LED_SK6812MINI_PLCC4_3.5x3.5mm_P1.75mm"
+		(property "Footprint" "Components:LED_SK6812MINI_PLCC4_3.5x3.5mm_P1.75mm"
 			(at 156.21 129.54 0)
 			(effects
