File: PCB/makropad.kicad_pcb (KiCad board)
At the start: 2 copper layers, 82 x 85 mm, 67 parts, among them J1 OLED_DISPLAY, J2 Conn_01x04, SW1 SW_Push_45deg, SW10 SW_Push_45deg, SW11 RotaryEncoder_Switch, SW12 RotaryEncoder_Switch, SW2 SW_Push_45deg, SW3 SW_Push_45deg, SW4 SW_Push_45deg, SW5 SW_Push_45deg, SW6 SW_Push_45deg, SW7 SW_Push_45deg, SW8 SW_Push_45deg, SW9 SW_Push_45deg, U1 PCF8574A, U2 MOUDLE-SEEEDUINO-XIAO

Commit message: feat: switch to choc v2 switches
Parts:
- D23, D24, D25, D26, D27, D28: footprint LED_SMD:LED_SK6812MINI_PLCC4_3.5x3.5mm_P1.75mm -> Components:LED_SK6812MINI_PLCC4_3.5x3.5mm_P1.75mm
- SW1, SW10, SW2, SW3, SW4, SW5, SW6, SW7, SW8, SW9: footprint Components:Gateron Low Profile Switch 2.0 -> Components:SW_Kailh_Choc_V2
- moved D4 19.6 mm to (190.0, 53.1)
- moved D8 19.5 mm to (189.9, 72.3)
- moved C10 14.6 mm to (168.0, 120.3), turned to 90 degrees
- moved C9 10.9 mm to (148.0, 120.4), turned to 90 degrees
- moved D21 10.1 mm to (142.9, 120.4)
- moved D22 10.1 mm to (162.0, 120.4)
- moved D15 10.1 mm to (162.1, 60.3)
- moved D19 10.1 mm to (162.1, 79.3)
- moved D13 10.1 mm to (124.0, 60.3)
- moved D14 10.1 mm to (143.0, 60.3)
- moved D16 10.1 mm to (181.1, 60.3)
- moved D17 10.1 mm to (124.0, 79.3)
- moved D18 10.1 mm to (143.0, 79.3)
- moved D20 10.1 mm to (181.1, 79.3)
- moved D2 10.0 mm to (152.0, 52.9)
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Routing:
- net GND: track 99.5 -> 165.9 mm, vias 50 -> 30
- net ROW1: track 51.9 -> 84.2 mm, vias 0 -> 2
- net ROW0: track 70.7 -> 101.3 mm
- net COL3: track 71.8 -> 96.2 mm
- net Net-(D20-DOUT): track 90.7 -> 71.7 mm, vias 2 -> 4
- net RGB: track 89.0 -> 70.4 mm, vias 0 -> 2
- net Net-(D11-A): track 20.5 -> 3.28 mm, vias 1 -> 0
- net COL1: track 112.3 -> 122.2 mm
- net STATUS_LED: track 78.5 -> 69.6 mm, vias 1 -> 2
- net COL0: track 130.6 -> 139.0 mm, vias 3 -> 2
- net Net-(D4-A): track 11.2 -> 3.95 mm
- net Net-(D8-A): track 11.1 -> 3.86 mm
- net COL2: track 89.9 -> 95.5 mm, vias 1 -> 0
- net Net-(D16-DOUT): track 88.4 -> 93.5 mm
- net Net-(D10-A): track 17.3 -> 13.9 mm
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
Commit message: Update production files
Routing:
- net ROW1: track 84.2 -> 84.8 mm
Changed lines of the file:
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@@
 	)
 	(segment
-		(start 180.84 86.313654)
-		(end 180.84 87.35)
+		(start 189.75 87.686346)
+		(end 188.936346 88.5)
 		(width 0.2)
 		(layer "F.Cu")
@@
 	)
 	(segment
-		(start 178.776346 84.25)
-		(end 180.84 86.313654)
+		(start 188.936346 88.5)
+		(end 181.99 88.5)
 		(width 0.2)
 		(layer "F.Cu")
@@
 	)
 	(segment
-		(start 170.9 73.95)
-		(end 170.9 76.632742)
+		(start 180.84 86.313654)
+		(end 180.84 87.35)
 		(width 0.2)
 		(layer "F.Cu")
@@
 	)
 	(segment
-		(start 189.75 87.686346)
-		(end 188.936346 88.5)
+		(start 178.776346 84.25)
+		(end 180.84 86.313654)
 		(width 0.2)
 		(layer "F.Cu")
@@
 	)
 	(segment
-		(start 188.936346 88.5)
-		(end 181.99 88.5)
+		(start 189.95 83.8)
+		(end 189.75 84)
 		(width 0.2)
 		(layer "F.Cu")
@@
 	)
 	(segment
-		(start 189.95 83.8)
-		(end 189.75 84)
+		(start 181.99 88.5)
+		(end 180.84 87.35)
 		(width 0.2)
 		(layer "F.Cu")
@@
 	)
 	(segment
-		(start 181.99 88.5)
-		(end 180.84 87.35)
+		(start 170.9 77.7)
+		(end 177.45 84.25)
 		(width 0.2)
 		(layer "F.Cu")
@@
 	)
 	(segment
-		(start 170.9 76.632742)
-		(end 178.517258 84.25)
+		(start 170.9 73.95)
+		(end 170.9 77.7)
 		(width 0.2)
 		(layer "F.Cu")
@@
 	)
 	(segment
-		(start 178.517258 84.25)
+		(start 177.45 84.25)
 		(end 178.776346 84.25)
 		(width 0.2)
@@
 	)
 	(segment
-		(start 123.95 70.354136)
-		(end 123.95 68.52)
-		(width 0.2)
-		(layer "F.Cu")
-		(net 24)
-	)
-	(segment
 		(start 138.32 93.15)
 		(end 137.25 94.22)
@@
 	)
 	(segment
-		(start 133.5 83.5)
-		(end 133.5 79.904136)
+		(start 138.52 92.95)
+		(end 138.52 88.52)
 		(width 0.2)
 		(layer "F.Cu")
@@
 	)
 	(segment
+		(start 138.52 88.52)
+		(end 133.5 83.5)
+		(width 0.2)
+		(layer "F.Cu")
+		(net 24)
+	)
+	(segment
+		(start 133.5 79.45)
+		(end 123.95 69.9)
+		(width 0.2)
+		(layer "F.Cu")
+		(net 24)
+	)
+	(segment
 		(start 137.25 94.22)
 		(end 137.25 108.5)
@@
 	)
 	(segment
-		(start 133.5 79.904136)
-		(end 123.95 70.354136)
+		(start 133.5 83.5)
+		(end 133.5 79.45)
 		(width 0.2)
 		(layer "F.Cu")
@@
 	)
 	(segment
-		(start 138.52 88.52)
-		(end 133.5 83.5)
+		(start 123.95 69.9)
+		(end 123.95 68.52)
 		(width 0.2)
 		(layer "F.Cu")
@@
 	)
 	(segment
-		(start 138.52 92.95)
-		(end 138.52 88.52)
-		(width 0.2)
-		(layer "F.Cu")
-		(net 24)
-	)
-	(segment
 		(start 120.75 52.67)
 		(end 123.95 49.47)
@@
 	)
 	(segment
-		(start 125.35 67.6)
+		(start 125.75 68)
 		(end 121.35 63.6)
 		(width 0.2)
@@
 	)
 	(segment
-		(start 125.35 71)
-		(end 125.35 67.6)
+		(start 134.1 82.45)
+		(end 134.1 79.15)
 		(width 0.2)
 		(layer "F.Cu")
@@
 	)
 	(segment
-		(start 134.1 79.75)
-		(end 125.35 71)
+		(start 134.1 79.15)
+		(end 125.75 70.8)
 		(width 0.2)
 		(layer "F.Cu")
@@
 	)
 	(segment
-		(start 134.1 82.45)
-		(end 134.1 79.75)
+		(start 125.75 70.8)
+		(end 125.75 68)
 		(width 0.2)
 		(layer "F.Cu")
